File: tiltbox.kicad_pcb (KiCad board)
At the start: 4 copper layers, 29 x 6.5 mm, 218 parts, among them J1 USB_C, J2 batt conn., SW1 SW_Wuerth_450301014042, U1 ESP32-C3-WROOM-02, U2 LIS2DH, U3 TP4056-42-ESOP8, U4 AMS1117-3.3

Commit message: i fixed the layout
Parts:
- moved C1 174.0 mm to (63.3, 74.4), turned to 0 degrees
- moved C11 171.3 mm to (63.3, 79.2), turned to 0 degrees
- moved LED91 170.6 mm to (58.1, 119.7)
- moved LED11 170.3 mm to (58.6, 81.5)
- moved LED31 170.2 mm to (58.6, 91.1)
- moved LED71 170.2 mm to (58.6, 110.3)
- moved C21 169.0 mm to (63.3, 84.0), turned to 0 degrees
- moved C91 167.9 mm to (63.0, 117.3), turned to 0 degrees
- moved C31 167.3 mm to (63.3, 88.8), turned to 0 degrees
- moved C81 166.3 mm to (63.3, 112.8), turned to 0 degrees
- moved C41 166.0 mm to (63.3, 93.6), turned to 0 degrees
- moved C71 165.4 mm to (63.3, 108.0), turned to 0 degrees
- moved C51 165.3 mm to (63.3, 98.4), turned to 0 degrees
- moved C2 165.2 mm to (68.1, 74.4)
- moved C61 165.1 mm to (63.3, 103.2), turned to 0 degrees
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- renumbered LED91 to LED100, LED20 to LED11, LED19 to LED12, LED18 to LED13, LED17 to LED14, LED16 to LED15, LED15 to LED16, LED14 to LED17, LED13 to LED18, LED12 to LED19, LED11 to LED20, LED40 to LED31, LED39 to LED32, LED38 to LED33, LED37 to LED34, LED36 to LED35, LED35 to LED36, LED34 to LED37, LED33 to LED38, LED32 to LED39, LED31 to LED40, LED60 to LED51, LED59 to LED52, LED58 to LED53, LED57 to LED54, LED56 to LED55, LED55 to LED56, LED54 to LED57, LED53 to LED58, LED52 to LED59, LED51 to LED60, LED80 to LED71, LED79 to LED72, LED78 to LED73, LED77 to LED74, LED76 to LED75, LED75 to LED76, LED74 to LED77, LED73 to LED78, LED72 to LED79, LED71 to LED80, LED100 to LED91, LED99 to LED92, LED98 to LED93, LED97 to LED94, LED96 to LED95, LED95 to LED96, LED94 to LED97, LED93 to LED98, LED92 to LED99
Routing:
- net +5V: track 0.00 -> 318.6 mm, vias 2 -> 103
- net Din_LED: track 0.00 -> 83.9 mm, vias 0 -> 1
- net battery output 5v: track 0.00 -> 50.9 mm, vias 0 -> 3
- net +3.3V: track 0.00 -> 44.7 mm
- net 5v output: track 0.00 -> 39.4 mm, vias 0 -> 1
- net Net-(D1-A): track 0.00 -> 38.9 mm, vias 0 -> 1
- net D+: track 0.00 -> 38.7 mm
- net D-: track 0.00 -> 34.5 mm
- net GND: track 0.00 -> 31.3 mm, vias 23 -> 212
- net Net-(U3-~{CHRG}): track 0.00 -> 29.3 mm
- net SDA: track 0.00 -> 25.9 mm
- net SCL: track 0.00 -> 22.5 mm
- net Net-(U3-~{STDBY}): track 0.00 -> 19.8 mm
- net Net-(LED51-DO): track 0.00 -> 5.55 mm
- net Net-(LED71-DO): track 0.00 -> 5.55 mm
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- added copper zone on In2.Cu, net +5V
- added copper zone on In1.Cu, net GND
- removed copper zone on In1.Cu, net +3.3V
- removed copper zone on In1.Cu, net +5V
- removed copper zone on In2.Cu, net GND
Other:
- board size 29 x 6.5 mm -> 69.3 x 69.4 mm
